File: mcr_shield.kicad_pcb (KiCad board)
At the start: 2 copper layers, 120 x 100 mm, 10 parts, among them J2 MCR_P1_Controls, J3 MCR_System_Coin, J4 MCR_Opt_X_Dial, J5 MCR_P2_Controls, SW1 Game_Selector, SW2 Cabinet_Options

Commit message: Add and route optocouplers, sync buffer, LM386 amp, and buck regulator to KiCad PCB file
Parts:
- added U1: Buck_Regulator, TO-220-3_Vertical, F.Cu at (115.0, 30.0)
- added U2: Optocoupler_P1, DIP-16_W7.62mm, F.Cu at (15.0, 45.0)
- added U3: Optocoupler_Sys, DIP-16_W7.62mm, F.Cu at (15.0, 65.0)
- added U4: Sync_Buffer, DIP-20_W7.62mm, F.Cu at (85.0, 30.0)
- added U5: Audio_Amplifier, DIP-8_W7.62mm, F.Cu at (115.0, 65.0)
Connections:
- J2 pad 1: BTN_LEFT -> CAB_BTN_LEFT
- J2 pad 2: BTN_RIGHT -> CAB_BTN_RIGHT
- J2 pad 5: BTN_FIRE -> CAB_BTN_FIRE
- J2 pad 6: BTN_SHIELD -> CAB_BTN_SHIELD
- J3 pad 1: BTN_COIN -> (no net)
- J3 pad 2: BTN_SERVICE -> (no net)
- J3 pad 3: BTN_START -> (no net)
- J3 pad 5: BTN_TILT -> (no net)
- JP1 pad 18: CAB_HS -> FPGA_HSYNC
- JP1 pad 19: CAB_VS -> FPGA_VSYNC
- JP1 pad 40: 12V_POWER -> 5V_REGULATED
- JP1 pad 5: BTN_START -> (no net)
- JP1 pad 6: BTN_COIN -> (no net)
- JP1 pad 7: BTN_SERVICE -> (no net)
- JP1 pad 8: BTN_TILT -> (no net)
- J_VID pad 8: CAB_HS -> CAB_HSYNC
- J_VID pad 9: CAB_VS -> CAB_VSYNC
